File: PCB_Electrical/projects/MURI_HASP_Integration/Relay_PCB.brd (EAGLE design)
At the start: 38.1 x 30.1 mm, 10 parts

Commit message: Added files for project schematics and boards that were developed this past summer
Parts:
- added H1, H2, H3, H4: MOUNT-HOLE3.0, holes:3,0
- moved SL3 6.35 mm to (44.5, 19.1)
- moved SL4 6.35 mm to (44.5, 27.9)
- moved SL1 5.08 mm to (0.00, 25.4)
Routing:
- net GND: track 66.6 -> 76.2 mm
- net OPC: track 20.1 -> 27.4 mm
- net OPC-ON: track 12.4 -> 18.7 mm
- net OPC-OFF: track 14.5 -> 20.8 mm
- net GOPRO-5V: track 40.0 -> 45.4 mm
Other:
- board size 38.1 x 30.1 mm -> 52.1 x 42.9 mm
