File: PCB_Electrical/projects/MURI_HASP_Integration/Relay_PCB.sch (EAGLE design)
At the start: 10 parts

Commit message: Added files for project schematics and boards that were developed this past summer
Parts:
- added H1, H2, H3, H4: MOUNT-HOLE3.0, holes:MOUNT-HOLE3.0
Changed lines of the file:
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@@
 <part name="SUPPLY5" library="supply2" library_urn="urn:adsk.eagle:library:372" deviceset="GND" device=""/>
 <part name="SUPPLY6" library="supply2" library_urn="urn:adsk.eagle:library:372" deviceset="GND" device=""/>
+<part name="H1" library="holes" deviceset="MOUNT-HOLE" device="3.0"/>
+<part name="H2" library="holes" deviceset="MOUNT-HOLE" device="3.0"/>
+<part name="H3" library="holes" deviceset="MOUNT-HOLE" device="3.0"/>
+<part name="H4" library="holes" deviceset="MOUNT-HOLE" device="3.0"/>
 </parts>
 <sheets>
@@
 <instance part="SUPPLY5" gate="GND" x="0" y="17.78"/>
 <instance part="SUPPLY6" gate="GND" x="106.68" y="43.18"/>
+<instance part="H1" gate="G$1" x="25.4" y="106.68"/>
+<instance part="H2" gate="G$1" x="91.44" y="106.68"/>
+<instance part="H3" gate="G$1" x="33.02" y="-12.7"/>
+<instance part="H4" gate="G$1" x="81.28" y="-10.16"/>
 </instances>
 <busses>
