File: PCB_Electrical/projects/MURI_HASP_Integration/Relay_PCB_v1.brd (EAGLE design)
At the start: 38.1 x 30.1 mm, 10 parts

Commit message: Added files for project schematics and boards that were developed this past summer
Parts:
- added H1, H2, H3, H4: MOUNT-HOLE3.0, holes:3,0
- moved SL3 8.89 mm to (47.0, 19.1)
- moved SL4 8.89 mm to (47.0, 27.9)
- moved SL1 5.08 mm to (0.00, 25.4)
Routing:
- net GND: track 66.6 -> 87.0 mm
- net OPC-ON: track 12.4 -> 21.3 mm
- net OPC-OFF: track 14.5 -> 23.4 mm
- net OPC: track 20.1 -> 28.8 mm
- net GOPRO-5V: track 40.0 -> 45.2 mm
- net N$3: track 11.6 -> 12.5 mm
Other:
- board size 38.1 x 30.1 mm -> 52 x 37.8 mm
