File: PCB_Electrical/projects/MURI_HASP_Integration/Relay_PCB_v1.sch (EAGLE design)
At the start: 10 parts

Commit message: Added files for project schematics and boards that were developed this past summer
Parts:
- added H1, H2, H3, H4: MOUNT-HOLE3.0, holes:MOUNT-HOLE3.0
Changed lines of the file:
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@@
 <class number="0" name="default" width="0" drill="0">
-</class>
-<class number="1" name="5V_Relay" width="0.254" drill="0.889">
-<clearance class="1" value="0.127"/>
 </class>
 </classes>
@@
 <part name="SUPPLY5" library="supply2" library_urn="urn:adsk.eagle:library:372" deviceset="GND" device=""/>
 <part name="SUPPLY6" library="supply2" library_urn="urn:adsk.eagle:library:372" deviceset="GND" device=""/>
+<part name="H1" library="holes" deviceset="MOUNT-HOLE" device="3.0"/>
+<part name="H2" library="holes" deviceset="MOUNT-HOLE" device="3.0"/>
+<part name="H3" library="holes" deviceset="MOUNT-HOLE" device="3.0"/>
+<part name="H4" library="holes" deviceset="MOUNT-HOLE" device="3.0"/>
 </parts>
 <sheets>
@@
 <instance part="SUPPLY5" gate="GND" x="0" y="17.78"/>
 <instance part="SUPPLY6" gate="GND" x="106.68" y="43.18"/>
+<instance part="H1" gate="G$1" x="38.1" y="101.6"/>
+<instance part="H2" gate="G$1" x="86.36" y="101.6"/>
+<instance part="H3" gate="G$1" x="40.64" y="0"/>
+<instance part="H4" gate="G$1" x="91.44" y="0"/>
 </instances>
 <busses>
 </busses>
 <nets>
-<net name="N$1" class="1">
+<net name="N$1" class="0">
 <segment>
 <pinref part="Q1" gate="G$1" pin="D"/>
@@
 </segment>
 </net>
-<net name="N$3" class="1">
+<net name="N$3" class="0">
 <segment>
 <pinref part="D2" gate="1" pin="A"/>
@@
 </segment>
 </net>
-<net name="GOPRO-5V" class="1">
+<net name="GOPRO-5V" class="0">
 <segment>
 <pinref part="D1" gate="1" pin="C"/>
@@
 </segment>
 </net>
-<net name="GND" class="1">
+<net name="GND" class="0">
 <segment>
 <pinref part="Q1" gate="G$1" pin="S"/>
@@
 </segment>
 </net>
-<net name="OPC-ON" class="1">
+<net name="OPC-ON" class="0">
 <segment>
 <pinref part="Q1" gate="G$1" pin="G"/>
@@
 </segment>
 </net>
-<net name="OPC-OFF" class="1">
+<net name="OPC-OFF" class="0">
 <segment>
 <pinref part="Q2" gate="G$1" pin="G"/>
@@
 </segment>
 </net>
-<net name="OPC" class="1">
+<net name="OPC" class="0">
 <segment>
 <pinref part="SL3" gate="G$1" pin="2"/>
